File: boards/alec-front/alec-front.kicad_sch (KiCad schematic)
At the start: 3 parts, among them J1 BM06B-GHS-TBT, SW1 BATTERY

Commit message: feat(rooster): consolidate the engineering baseline (#129)
* docs(rooster): start prototype order preparation and sourcing inventory

* docs(rooster): record JLCPCB quantities and assembly-side preflight

* docs(rooster): distinguish Beacon radar module from assembly socket

* feat(rooster): prepare sourced prototype BOM and complete placement drafts

* feat(rooster): validate prototype power parts and refine capacitor sourcing

* fix(rooster): synchronize assembly selections with native board sources

* feat(rooster): verify fabrication candidates and start supplier quote

* docs(rooster): require explicit approval before purchasing

* docs(rooster): record assembly quote and RTC sourcing options

* fix(rooster): correct controls placement centers and capture assembly quotes

* fix(rooster): correct header placements and capture four-board estimates

* docs(rooster): resolve amplifier copper pattern and stage production review

* docs(rooster): record LED fuse and header review findings

* docs(rooster): specify capped vias and verify mask clearance

* docs(rooster): verify mask bridges and prepare exact RTC preorder

* fix(rooster): allow finished-hole tolerance at main display header

* fab(rooster): export checked header-fit candidates and rebind placements

* Bind prototype via process attachments to current fabrication files

* Define prototype stackup and record USB functional-test disposition

* Record updated main quote with current Gerbers and fill-cap stackup

* docs(rooster): refresh Beacon quote and first-power handoff

* docs(rooster): prepare exact placement review and external inventory

* docs(rooster): define immediate order gates and prototype power scope

* docs(rooster): compare stocked RTC alternatives and compatibility

* docs(rooster): compare RTC manufacturers and enclosure thermal limits

* docs(rooster): compare PCB manufacturing and assembly suppliers

* docs(rooster): stage Cube first and retain JLCPCB recommendation

* docs(rooster): re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
Parts:
- D1: LCSC# (none) -> C5342281; Manufacturer (none) -> Wurth Elektronik
- J1: LCSC# (none) -> C189892; MPN BM06B-GHS-TBT -> BM06B-GHS-TBT(LF)(SN); Manufacturer (none) -> JST
- SW1: LCSC# (none) -> C231329; Manufacturer (none) -> Omron Electronics
Changed lines of the file:
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@@
 		(property
 			"MPN"
-			"BM06B-GHS-TBT"
+			"BM06B-GHS-TBT(LF)(SN)"
 			(at 49.53 64.77 0)
 			(effects
@@
 		(pin
 			"6"
-))
+)
+	(property "Manufacturer" "JST" (at 0 0 0) (effects (font (size 1.27 1.27)) (hide yes)))
+	(property "LCSC#" "C189892" (at 0 0 0) (effects (font (size 1.27 1.27)) (hide yes))))
 	(wire
 		(pts
@@
 		(pin
 			"2"
-))
+)
+	(property "Manufacturer" "Omron Electronics" (at 0 0 0) (effects (font (size 1.27 1.27)) (hide yes)))
+	(property "LCSC#" "C231329" (at 0 0 0) (effects (font (size 1.27 1.27)) (hide yes))))
 	(wire
 		(pts
@@
 		(pin
 			"1"
-))
+)
+	(property "Manufacturer" "Wurth Elektronik" (at 0 0 0) (effects (font (size 1.27 1.27)) (hide yes)))
+	(property "LCSC#" "C5342281" (at 0 0 0) (effects (font (size 1.27 1.27)) (hide yes))))
 	(text
 		"1:1 GH harness to main J6; LED series resistors on main"
