File: boards/alec-main/alec-main.kicad_sch (KiCad schematic)
At the start: 98 parts, among them J1 Conn_01x02_Pin, J2 USB_C_Receptacle_USB2.0_16P, J3 Conn_01x02_Pin, J4 Conn_01x04_Pin, J5 BM07B-GHS-TBT, J6 BM06B-GHS-TBT, J7 UNPOPULATED_TEST_PADS, Q1 AO3401A, Q2 AO3401A, Q3 MMBT3904, SW2 RESET, SW3 BOOT, U1 TPS63070RNMR, U2 TPS63070RNMR, U3 ESP32-S3-WROOM-1-N16, U4 USBLC6-2SC6, U5 RV-3028-C7, U6 MAX98357A, U7 SN74LVC2G66DCUR, U8 SN74LVC1T45DBVR

Commit message: feat(rooster): consolidate the engineering baseline (#129)
* docs(rooster): start prototype order preparation and sourcing inventory

* docs(rooster): record JLCPCB quantities and assembly-side preflight

* docs(rooster): distinguish Beacon radar module from assembly socket

* feat(rooster): prepare sourced prototype BOM and complete placement drafts

* feat(rooster): validate prototype power parts and refine capacitor sourcing

* fix(rooster): synchronize assembly selections with native board sources

* feat(rooster): verify fabrication candidates and start supplier quote

* docs(rooster): require explicit approval before purchasing

* docs(rooster): record assembly quote and RTC sourcing options

* fix(rooster): correct controls placement centers and capture assembly quotes

* fix(rooster): correct header placements and capture four-board estimates

* docs(rooster): resolve amplifier copper pattern and stage production review

* docs(rooster): record LED fuse and header review findings

* docs(rooster): specify capped vias and verify mask clearance

* docs(rooster): verify mask bridges and prepare exact RTC preorder

* fix(rooster): allow finished-hole tolerance at main display header

* fab(rooster): export checked header-fit candidates and rebind placements

* Bind prototype via process attachments to current fabrication files

* Define prototype stackup and record USB functional-test disposition

* Record updated main quote with current Gerbers and fill-cap stackup

* docs(rooster): refresh Beacon quote and first-power handoff

* docs(rooster): prepare exact placement review and external inventory

* docs(rooster): define immediate order gates and prototype power scope

* docs(rooster): compare stocked RTC alternatives and compatibility

* docs(rooster): compare RTC manufacturers and enclosure thermal limits

* docs(rooster): compare PCB manufacturing and assembly suppliers

* docs(rooster): stage Cube first and retain JLCPCB recommendation

* docs(rooster): re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
Parts:
- C1, C10, C2, C27, C9: LCSC# (none) -> C84416; MPN (none) -> GRM21BR61E106KA73L; Manufacturer (none) -> Murata Electronics
- C11, C13, C3, C5: LCSC# (none) -> C782172; MPN (none) -> GRT188R61A106KE13D; Manufacturer (none) -> Murata Electronics
- C12, C18, C20, C22, C23, C24, C25, C28, C29, C30, C32, C33, C4: LCSC# (none) -> C71629; MPN (none) -> GRM155R71C104KA88D; Manufacturer (none) -> Murata Electronics
- C14, C15, C16, C6, C7, C8: LCSC# (none) -> C77088; Manufacturer (none) -> Murata Electronics
- C17: LCSC# (none) -> C441864; MPN (none) -> GRM21BR61A226ME44L; Manufacturer (none) -> Murata Electronics
- C19: LCSC# (none) -> C76999; MPN (none) -> GRM155R61A105KE15D; Manufacturer (none) -> Murata Electronics
- C21, C26: LCSC# (none) -> C883598; MPN (none) -> GRM31CR61A107MEA8L; Manufacturer (none) -> Murata Electronics
- C31: LCSC# (none) -> C86012; MPN (none) -> GRM188R61A105KA61D; Manufacturer (none) -> Murata Electronics
- D1: LCSC# (none) -> C125094; MPN (none) -> LTST-C190KGKT; Manufacturer (none) -> Lite-On
- J1, J3: LCSC# (none) -> C160352; MPN (none) -> B2B-PH-SM4-TB(LF)(SN); Manufacturer (none) -> JST
- J2: LCSC# (none) -> C165948; MPN (none) -> TYPE-C-31-M-12; Manufacturer (none) -> Korean Hroparts Elec
- J4: footprint Connector_PinHeader_2.54mm:PinHeader_1x04_P2.54mm_Vertical -> Board:Samtec_TSW-104-07-G-S_Drill1.10mm; LCSC# (none) -> C3335156; MPN (none) -> TSW-104-07-G-S; Manufacturer (none) -> Samtec
- J5: LCSC# (none) -> C5305068; MPN BM07B-GHS-TBT -> BM07B-GHS-TBT(LF)(SN); Manufacturer (none) -> JST
- J6: LCSC# (none) -> C189892; MPN BM06B-GHS-TBT -> BM06B-GHS-TBT(LF)(SN); Manufacturer (none) -> JST
- L1, L2: LCSC# (none) -> C3033018; Manufacturer (none) -> Coilcraft
- Q1, Q2: LCSC# (none) -> C15127; MPN (none) -> AO3401A; Manufacturer (none) -> Alpha & Omega Semicon
- Q3: LCSC# (none) -> C81464; MPN (none) -> MMBT3904LT1G; Manufacturer (none) -> onsemi
- R1, R10, R19, R20, R21, R23, R32, R36, R39, R6: LCSC# (none) -> C60491; MPN (none) -> RC0402FR-07100KL; Manufacturer (none) -> YAGEO
- R12, R13, R18, R22, R24, R25, R26, R27, R3, R31, R33, R7: LCSC# (none) -> C60490; MPN (none) -> RC0402FR-0710KL; Manufacturer (none) -> YAGEO
- R14, R15: LCSC# (none) -> C105872; MPN (none) -> RC0402FR-075K1L; Manufacturer (none) -> YAGEO
- R16, R17, R37, R38: LCSC# (none) -> C105871; MPN (none) -> RC0402FR-074K7L; Manufacturer (none) -> YAGEO
- R28: LCSC# (none) -> C105875; MPN (none) -> RC0402FR-07330RL; Manufacturer (none) -> YAGEO
- R29, R30: LCSC# (none) -> C25082; MPN (none) -> 0402WGF1500TCE; Manufacturer (none) -> UNI-ROYAL(Uniroyal Elec)
- R34, R35: LCSC# (none) -> C114765; MPN (none) -> RC0402FR-0722RL; Manufacturer (none) -> YAGEO
- R4: LCSC# (none) -> C137976; MPN (none) -> RC0402FR-07470KL; Manufacturer (none) -> YAGEO
- R5: LCSC# (none) -> C93947; MPN (none) -> RC0402FR-07150KL; Manufacturer (none) -> YAGEO
- R50, R51, R52, R53: LCSC# (none) -> C106232; Manufacturer (none) -> YAGEO
- R8: LCSC# (none) -> C163456; MPN (none) -> RC0402FR-07680KL; Manufacturer (none) -> YAGEO
- R9: LCSC# (none) -> C93946; MPN (none) -> RC0402FR-07130KL; Manufacturer (none) -> YAGEO
- SW2, SW3: LCSC# (none) -> C318884; MPN (none) -> TS-1187A-B-A-B; Manufacturer (none) -> XKB Connection
- U1, U2: LCSC# (none) -> C109322; MPN (none) -> TPS63070RNMR; Manufacturer (none) -> Texas Instruments
- U3: LCSC# (none) -> C2913199; MPN (none) -> ESP32-S3-WROOM-1-N16; Manufacturer (none) -> Espressif Systems
- U4: LCSC# (none) -> C7519; MPN (none) -> USBLC6-2SC6; Manufacturer (none) -> STMicroelectronics
- U5: LCSC# (none) -> C3019759; MPN (none) -> RV-3028-C7-32.768kHz-1ppm-TA-QC; Manufacturer (none) -> Micro Crystal
- U6: LCSC# (none) -> C910544; MPN (none) -> MAX98357AETE+T; Manufacturer (none) -> Analog Devices Inc./Maxim Integrated
- U7: LCSC# (none) -> C181970; MPN (none) -> SN74LVC2G66DCUR; Manufacturer (none) -> Texas Instruments
- U8: LCSC# (none) -> C7843; MPN (none) -> SN74LVC1T45DBVR; Manufacturer (none) -> Texas Instruments
