File: boards/alec-main/power-monitor.kicad_sch (KiCad schematic)
At the start: 15 parts, among them Q4 MMBT3904, Q5 MMBT3904, Q6 AO3401A, Q7 MMBT3904

Commit message: feat(rooster): consolidate the engineering baseline (#129)
* docs(rooster): start prototype order preparation and sourcing inventory

* docs(rooster): record JLCPCB quantities and assembly-side preflight

* docs(rooster): distinguish Beacon radar module from assembly socket

* feat(rooster): prepare sourced prototype BOM and complete placement drafts

* feat(rooster): validate prototype power parts and refine capacitor sourcing

* fix(rooster): synchronize assembly selections with native board sources

* feat(rooster): verify fabrication candidates and start supplier quote

* docs(rooster): require explicit approval before purchasing

* docs(rooster): record assembly quote and RTC sourcing options

* fix(rooster): correct controls placement centers and capture assembly quotes

* fix(rooster): correct header placements and capture four-board estimates

* docs(rooster): resolve amplifier copper pattern and stage production review

* docs(rooster): record LED fuse and header review findings

* docs(rooster): specify capped vias and verify mask clearance

* docs(rooster): verify mask bridges and prepare exact RTC preorder

* fix(rooster): allow finished-hole tolerance at main display header

* fab(rooster): export checked header-fit candidates and rebind placements

* Bind prototype via process attachments to current fabrication files

* Define prototype stackup and record USB functional-test disposition

* Record updated main quote with current Gerbers and fill-cap stackup

* docs(rooster): refresh Beacon quote and first-power handoff

* docs(rooster): prepare exact placement review and external inventory

* docs(rooster): define immediate order gates and prototype power scope

* docs(rooster): compare stocked RTC alternatives and compatibility

* docs(rooster): compare RTC manufacturers and enclosure thermal limits

* docs(rooster): compare PCB manufacturing and assembly suppliers

* docs(rooster): stage Cube first and retain JLCPCB recommendation

* docs(rooster): re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
Parts:
- C34: LCSC# (none) -> C71629; MPN (none) -> GRM155R71C104KA88D; Manufacturer (none) -> Murata Electronics
- Q4, Q5, Q7: LCSC# (none) -> C81464; MPN (none) -> MMBT3904LT1G; Manufacturer (none) -> onsemi
- Q6: LCSC# (none) -> C15127; MPN (none) -> AO3401A; Manufacturer (none) -> Alpha & Omega Semicon
- R40, R45, R47: LCSC# (none) -> C60491; MPN (none) -> RC0402FR-07100KL; Manufacturer (none) -> YAGEO
- R41: LCSC# (none) -> C138033; MPN (none) -> RC0402FR-071ML; Manufacturer (none) -> YAGEO
- R42, R44: LCSC# (none) -> C93943; MPN (none) -> RC0402FR-0747KL; Manufacturer (none) -> YAGEO
- R43, R46: LCSC# (none) -> C60490; MPN (none) -> RC0402FR-0710KL; Manufacturer (none) -> YAGEO
- R48: LCSC# (none) -> C728559; Manufacturer (none) -> YAGEO
- R49: LCSC# (none) -> C190095; Manufacturer (none) -> YAGEO
