File: boards/alec-sensor/alec-sensor.kicad_sch (KiCad schematic)
At the start: 65 parts, among them J1 Conn_01x02_Pin, J2 USB_C_Receptacle_USB2.0_16P, Q1 AO3401A, SW1 1101M2S3CQE2, SW2 RESET, SW3 BOOT, SW7 BATTERY / PAIR, U1 TPS63070RNMR, U2 TPS63070RNMR, U3 ESP32-S3-WROOM-1-N16, U4 USBLC6-2SC6, U5 RV-3028-C7

Commit message: feat(rooster): consolidate the engineering baseline (#129)
* docs(rooster): start prototype order preparation and sourcing inventory

* docs(rooster): record JLCPCB quantities and assembly-side preflight

* docs(rooster): distinguish Beacon radar module from assembly socket

* feat(rooster): prepare sourced prototype BOM and complete placement drafts

* feat(rooster): validate prototype power parts and refine capacitor sourcing

* fix(rooster): synchronize assembly selections with native board sources

* feat(rooster): verify fabrication candidates and start supplier quote

* docs(rooster): require explicit approval before purchasing

* docs(rooster): record assembly quote and RTC sourcing options

* fix(rooster): correct controls placement centers and capture assembly quotes

* fix(rooster): correct header placements and capture four-board estimates

* docs(rooster): resolve amplifier copper pattern and stage production review

* docs(rooster): record LED fuse and header review findings

* docs(rooster): specify capped vias and verify mask clearance

* docs(rooster): verify mask bridges and prepare exact RTC preorder

* fix(rooster): allow finished-hole tolerance at main display header

* fab(rooster): export checked header-fit candidates and rebind placements

* Bind prototype via process attachments to current fabrication files

* Define prototype stackup and record USB functional-test disposition

* Record updated main quote with current Gerbers and fill-cap stackup

* docs(rooster): refresh Beacon quote and first-power handoff

* docs(rooster): prepare exact placement review and external inventory

* docs(rooster): define immediate order gates and prototype power scope

* docs(rooster): compare stocked RTC alternatives and compatibility

* docs(rooster): compare RTC manufacturers and enclosure thermal limits

* docs(rooster): compare PCB manufacturing and assembly suppliers

* docs(rooster): stage Cube first and retain JLCPCB recommendation

* docs(rooster): re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
Parts:
- C1, C10, C2, C9: LCSC# (none) -> C84416; Manufacturer (none) -> Murata Electronics
- C11, C13, C3, C5: LCSC# (none) -> C782172; MPN GRM188R61A106KAALD -> GRT188R61A106KE13D; Manufacturer (none) -> Murata Electronics
- C12, C18, C20, C25, C29, C4: LCSC# (none) -> C71629; Manufacturer (none) -> Murata Electronics
- C14, C15, C16, C6, C7, C8: LCSC# (none) -> C77088; Manufacturer (none) -> Murata Electronics
- C17: LCSC# (none) -> C441864; Manufacturer (none) -> Murata Electronics
- C19: LCSC# (none) -> C76999; Manufacturer (none) -> Murata Electronics
- C21: LCSC# (none) -> C15008; Manufacturer (none) -> Samsung Electro-Mechanics
- D2: LCSC# (none) -> C5342281; Manufacturer (none) -> Wurth Elektronik
- F1: LCSC# (none) -> C187608; Manufacturer (none) -> Littelfuse
- J1: LCSC# (none) -> C160352; Manufacturer (none) -> JST
- J2: LCSC# (none) -> C165948; Manufacturer (none) -> Korean Hroparts Elec
- L1, L2: LCSC# (none) -> C3033018; Manufacturer (none) -> Coilcraft
- Q1: LCSC# (none) -> C15127; Manufacturer (none) -> Alpha & Omega Semicon
- R1, R10, R19, R32, R6: LCSC# (none) -> C60491; Manufacturer (none) -> YAGEO
- R12, R13, R18, R27, R3, R31, R33, R7: LCSC# (none) -> C60490; Manufacturer (none) -> YAGEO
- R14, R15: LCSC# (none) -> C105872; Manufacturer (none) -> YAGEO
- R16, R17: LCSC# (none) -> C105871; Manufacturer (none) -> YAGEO
- R28: LCSC# (none) -> C105875; Manufacturer (none) -> YAGEO
- R29, R30: LCSC# (none) -> C25082; MPN RC0402FR-07150RL -> 0402WGF1500TCE; Manufacturer (none) -> UNI-ROYAL(Uniroyal Elec)
- R34, R35: LCSC# (none) -> C114765; Manufacturer (none) -> YAGEO
- R4: LCSC# (none) -> C137976; Manufacturer (none) -> YAGEO
- R5: LCSC# (none) -> C93947; Manufacturer (none) -> YAGEO
- R8: LCSC# (none) -> C163456; Manufacturer (none) -> YAGEO
- R9: LCSC# (none) -> C93946; Manufacturer (none) -> YAGEO
- SW1: LCSC# (none) -> C221538; Manufacturer (none) -> C&K
- SW2, SW3, SW7: LCSC# (none) -> C318884; Manufacturer (none) -> XKB Connection
- U1, U2: LCSC# (none) -> C109322; Manufacturer (none) -> Texas Instruments
- U3: LCSC# (none) -> C2913199; Manufacturer (none) -> Espressif Systems
- U4: LCSC# (none) -> C7519; Manufacturer (none) -> STMicroelectronics
- U5: LCSC# (none) -> C3019759; MPN RV-3028-C7 -> RV-3028-C7-32.768kHz-1ppm-TA-QC; Manufacturer (none) -> Micro Crystal
