File: boards/alec-sensor/power-monitor.kicad_sch (KiCad schematic)
At the start: 15 parts, among them Q4 MMBT3904, Q5 MMBT3904, Q6 AO3401A, Q7 MMBT3904

Commit message: feat(rooster): consolidate the engineering baseline (#129)
* docs(rooster): start prototype order preparation and sourcing inventory

* docs(rooster): record JLCPCB quantities and assembly-side preflight

* docs(rooster): distinguish Beacon radar module from assembly socket

* feat(rooster): prepare sourced prototype BOM and complete placement drafts

* feat(rooster): validate prototype power parts and refine capacitor sourcing

* fix(rooster): synchronize assembly selections with native board sources

* feat(rooster): verify fabrication candidates and start supplier quote

* docs(rooster): require explicit approval before purchasing

* docs(rooster): record assembly quote and RTC sourcing options

* fix(rooster): correct controls placement centers and capture assembly quotes

* fix(rooster): correct header placements and capture four-board estimates

* docs(rooster): resolve amplifier copper pattern and stage production review

* docs(rooster): record LED fuse and header review findings

* docs(rooster): specify capped vias and verify mask clearance

* docs(rooster): verify mask bridges and prepare exact RTC preorder

* fix(rooster): allow finished-hole tolerance at main display header

* fab(rooster): export checked header-fit candidates and rebind placements

* Bind prototype via process attachments to current fabrication files

* Define prototype stackup and record USB functional-test disposition

* Record updated main quote with current Gerbers and fill-cap stackup

* docs(rooster): refresh Beacon quote and first-power handoff

* docs(rooster): prepare exact placement review and external inventory

* docs(rooster): define immediate order gates and prototype power scope

* docs(rooster): compare stocked RTC alternatives and compatibility

* docs(rooster): compare RTC manufacturers and enclosure thermal limits

* docs(rooster): compare PCB manufacturing and assembly suppliers

* docs(rooster): stage Cube first and retain JLCPCB recommendation

* docs(rooster): re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
Parts:
- C34: LCSC# (none) -> C71629; Manufacturer (none) -> Murata Electronics
- Q4, Q5, Q7: LCSC# (none) -> C81464; MPN MMBT3904 -> MMBT3904LT1G; Manufacturer (none) -> onsemi
- Q6: LCSC# (none) -> C15127; Manufacturer (none) -> Alpha & Omega Semicon
- R40, R45, R47: LCSC# (none) -> C60491; Manufacturer (none) -> YAGEO
- R41: LCSC# (none) -> C138033; Manufacturer (none) -> YAGEO
- R42, R44: LCSC# (none) -> C93943; Manufacturer (none) -> YAGEO
- R43, R46: LCSC# (none) -> C60490; Manufacturer (none) -> YAGEO
- R48: LCSC# (none) -> C728559; Manufacturer (none) -> YAGEO
- R49: LCSC# (none) -> C190095; Manufacturer (none) -> YAGEO
Changed lines of the file:
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@@
 		(property
 			"MPN"
-			"MMBT3904"
+			"MMBT3904LT1G"
 			(at 0 0 0)
 			(effects
 				(font
 					(size 1.27 1.27))
-				(hide yes))))
+				(hide yes)))
+	(property "Manufacturer" "onsemi" (at 0 0 0) (effects (font (size 1.27 1.27)) (hide yes)))
+	(property "LCSC#" "C81464" (at 0 0 0) (effects (font (size 1.27 1.27)) (hide yes))))
 	(symbol
 		(lib_id "Transistor_BJT:MMBT3904")
@@
 		(property
 			"MPN"
-			"MMBT3904"
+			"MMBT3904LT1G"
 			(at 0 0 0)
 			(effects
 				(font
 					(size 1.27 1.27))
-				(hide yes))))
+				(hide yes)))
+	(property "Manufacturer" "onsemi" (at 0 0 0) (effects (font (size 1.27 1.27)) (hide yes)))
+	(property "LCSC#" "C81464" (at 0 0 0) (effects (font (size 1.27 1.27)) (hide yes))))
 	(symbol
 		(lib_id "Device:R")
@@
 		(property
 			"Datasheet"
-			"https://www.yageo.com/en/Product/Index/rchip/rc"
+			"https://www.lcsc.com/datasheet/lcsc_datasheet_2304140030_YAGEO-RC0402FR-07100KL_C60491.pdf"
 			(at 45.72 66.04 0)
 			(hide yes)
@@
 				(font
 					(size 1.27 1.27))
-				(hide yes))))
+				(hide yes)))
+	(property "Manufacturer" "YAGEO" (at 0 0 0) (effects (font (size 1.27 1.27)) (hide yes)))
+	(property "LCSC#" "C60491" (at 0 0 0) (effects (font (size 1.27 1.27)) (hide yes))))
 	(symbol
 		(lib_id "Device:R")
@@
 		(property
 			"Datasheet"
-			"https://www.yageo.com/en/Product/Index/rchip/rc"
+			"https://www.lcsc.com/datasheet/lcsc_datasheet_2304140030_YAGEO-RC0402FR-071ML_C138033.pdf"
 			(at 53.34 82.55 0)
 			(hide yes)
@@
 				(font
 					(size 1.27 1.27))
-				(hide yes))))
+				(hide yes)))
+	(property "Manufacturer" "YAGEO" (at 0 0 0) (effects (font (size 1.27 1.27)) (hide yes)))
+	(property "LCSC#" "C138033" (at 0 0 0) (effects (font (size 1.27 1.27)) (hide yes))))
 	(symbol
 		(lib_id "Device:R")
@@
 		(property
 			"Datasheet"
-			"https://www.yageo.com/en/Product/Index/rchip/rc"
+			"https://www.lcsc.com/datasheet/lcsc_datasheet_2304140030_YAGEO-RC0402FR-0747KL_C93943.pdf"
 			(at 66.04 48.26 0)
 			(hide yes)
@@
 				(font
 					(size 1.27 1.27))
-				(hide yes))))
+				(hide yes)))
+	(property "Manufacturer" "YAGEO" (at 0 0 0) (effects (font (size 1.27 1.27)) (hide yes)))
+	(property "LCSC#" "C93943" (at 0 0 0) (effects (font (size 1.27 1.27)) (hide yes))))
 	(symbol
 		(lib_id "Device:R")
@@
 		(property
 			"Datasheet"
-			"https://www.yageo.com/en/Product/Index/rchip/rc"
+			"https://www.lcsc.com/datasheet/lcsc_datasheet_2304140030_YAGEO-RC0402FR-0710KL_C60490.pdf"
 			(at 91.44 66.04 0)
 			(hide yes)
@@
 				(font
 					(size 1.27 1.27))
-				(hide yes))))
+				(hide yes)))
+	(property "Manufacturer" "YAGEO" (at 0 0 0) (effects (font (size 1.27 1.27)) (hide yes)))
+	(property "LCSC#" "C60490" (at 0 0 0) (effects (font (size 1.27 1.27)) (hide yes))))
 	(symbol
 		(lib_id "Device:R")
@@
 		(property
 			"Datasheet"
-			"https://www.yageo.com/en/Product/Index/rchip/rc"
+			"https://www.lcsc.com/datasheet/lcsc_datasheet_2304140030_YAGEO-RC0402FR-0747KL_C93943.pdf"
 			(at 116.84 48.26 0)
 			(hide yes)
@@
 				(font
 					(size 1.27 1.27))
-				(hide yes))))
+				(hide yes)))
+	(property "Manufacturer" "YAGEO" (at 0 0 0) (effects (font (size 1.27 1.27)) (hide yes)))
+	(property "LCSC#" "C93943" (at 0 0 0) (effects (font (size 1.27 1.27)) (hide yes))))
 	(wire
 		(pts
@@
 		(property
 			"Datasheet"
-			"https://www.aosmd.com/sites/default/files/res/datasheets/AO3401A.pdf"
+			"https://www.lcsc.com/datasheet/lcsc_datasheet_2412061733_Alpha---Omega-Semicon-AO3401A_C15127.pdf"
 			(at 88.9 147.32 0)
 			(hide yes)
@@
 				(font
 					(size 1.27 1.27))
-				(hide yes))))
+				(hide yes)))
+	(property "Manufacturer" "Alpha & Omega Semicon" (at 0 0 0) (effects (font (size 1.27 1.27)) (hide yes)))
+	(property "LCSC#" "C15127" (at 0 0 0) (effects (font (size 1.27 1.27)) (hide yes))))
 	(symbol
 		(lib_id "Device:R")
@@
 		(property
 			"Datasheet"
-			"https://www.yageo.com/en/Product/Index/rchip/rc"
+			"https://www.lcsc.com/datasheet/lcsc_datasheet_2304140030_YAGEO-RC0402FR-07100KL_C60491.pdf"
 			(at 106.68 138.43 0)
 			(hide yes)
@@
 				(font
 					(size 1.27 1.27))
-				(hide yes))))
+				(hide yes)))
+	(property "Manufacturer" "YAGEO" (at 0 0 0) (effects (font (size 1.27 1.27)) (hide yes)))
+	(property "LCSC#" "C60491" (at 0 0 0) (effects (font (size 1.27 1.27)) (hide yes))))
 	(symbol
 		(lib_id "Transistor_BJT:MMBT3904")
@@
 		(property
 			"MPN"
-			"MMBT3904"
+			"MMBT3904LT1G"
 			(at 0 0 0)
 			(effects
 				(font
 					(size 1.27 1.27))
-				(hide yes))))
+				(hide yes)))
+	(property "Manufacturer" "onsemi" (at 0 0 0) (effects (font (size 1.27 1.27)) (hide yes)))
+	(property "LCSC#" "C81464" (at 0 0 0) (effects (font (size 1.27 1.27)) (hide yes))))
 	(symbol
 		(lib_id "Device:R")
@@
 		(property
 			"Datasheet"
-			"https://www.yageo.com/en/Product/Index/rchip/rc"
+			"https://www.lcsc.com/datasheet/lcsc_datasheet_2304140030_YAGEO-RC0402FR-0710KL_C60490.pdf"
 			(at 99.06 165.1 0)
 			(hide yes)
@@
 				(font
 					(size 1.27 1.27))
-				(hide yes))))
+				(hide yes)))
+	(property "Manufacturer" "YAGEO" (at 0 0 0) (effects (font (size 1.27 1.27)) (hide yes)))
+	(property "LCSC#" "C60490" (at 0 0 0) (effects (font (size 1.27 1.27)) (hide yes))))
 	(symbol
 		(lib_id "Device:R")
@@
 		(property
 			"Datasheet"
-			"https://www.yageo.com/en/Product/Index/rchip/rc"
+			"https://www.lcsc.com/datasheet/lcsc_datasheet_2304140030_YAGEO-RC0402FR-07100KL_C60491.pdf"
 			(at 109.22 179.07 0)
 			(hide yes)
@@
 				(font
 					(size 1.27 1.27))
-				(hide yes))))
+				(hide yes)))
+	(property "Manufacturer" "YAGEO" (at 0 0 0) (effects (font (size 1.27 1.27)) (hide yes)))
+	(property "LCSC#" "C60491" (at 0 0 0) (effects (font (size 1.27 1.27)) (hide yes))))
 	(symbol
 		(lib_id "Device:R")
@@
 		(property
 			"Datasheet"
-			""
+			"https://wmsc.lcsc.com/wmsc/upload/file/pdf/v2/lcsc/2304140030_YAGEO-RT0402BRD0733KL_C728559.pdf"
 			(at 132.07999999999998 149.86 0)
 			(hide yes)
@@
 					"/7924bd8b-2498-4d76-899d-c0ad5a514485/7c84093a-5796-4504-a572-6cccb77c9bc7"
 					(reference "R48")
-					(unit 1)))))
+					(unit 1))))
+	(property "Manufacturer" "YAGEO" (at 0 0 0) (effects (font (size 1.27 1.27)) (hide yes)))
+	(property "LCSC#" "C728559" (at 0 0 0) (effects (font (size 1.27 1.27)) (hide yes))))
 	(symbol
 		(lib_id "Device:R")
@@
 		(property
 			"Datasheet"
-			""
+			"https://www.lcsc.com/datasheet/lcsc_datasheet_2304140030_YAGEO-RT0402BRD0710KL_C190095.pdf"
 			(at 132.07999999999998 175.26 0)
 			(hide yes)
@@
 					"/7924bd8b-2498-4d76-899d-c0ad5a514485/7c84093a-5796-4504-a572-6cccb77c9bc7"
 					(reference "R49")
-					(unit 1)))))
+					(unit 1))))
+	(property "Manufacturer" "YAGEO" (at 0 0 0) (effects (font (size 1.27 1.27)) (hide yes)))
+	(property "LCSC#" "C190095" (at 0 0 0) (effects (font (size 1.27 1.27)) (hide yes))))
 	(symbol
 		(lib_id "Device:C")
@@
 		(property
 			"Datasheet"
-			"https://search.murata.co.jp/Ceramy/image/img/A01X/G101/ENG/GRM155R71C104KA88-01A.pdf"
+			"https://www.lcsc.com/datasheet/lcsc_datasheet_1811081616_Murata-Electronics-GRM155R71C104KA88D_C71629.pdf"
 			(at 154.94 175.26 0)
 			(hide yes)
@@
 				(font
 					(size 1.27 1.27))
-				(hide yes))))
-	(wire
-		(pts
+				(hide yes)))
+	(property "Manufacturer" "Murata Electronics" (at 0 0 0) (effects (font (size 1.27 1.27)) (hide yes)))
+	(property "LCSC#" "C71629" (at 0 0 0) (effects (font (size 1.27 1.27)) (hide yes))))
+	(wire
+		(pts
