File: boards/alec-sensor/radar.kicad_sch (KiCad schematic)
At the start: 8 parts, among them J3 LD2410C — INTERNAL, U10 TMUX1511PWR

Commit message: feat(rooster): consolidate the engineering baseline (#129)
* docs(rooster): start prototype order preparation and sourcing inventory

* docs(rooster): record JLCPCB quantities and assembly-side preflight

* docs(rooster): distinguish Beacon radar module from assembly socket

* feat(rooster): prepare sourced prototype BOM and complete placement drafts

* feat(rooster): validate prototype power parts and refine capacitor sourcing

* fix(rooster): synchronize assembly selections with native board sources

* feat(rooster): verify fabrication candidates and start supplier quote

* docs(rooster): require explicit approval before purchasing

* docs(rooster): record assembly quote and RTC sourcing options

* fix(rooster): correct controls placement centers and capture assembly quotes

* fix(rooster): correct header placements and capture four-board estimates

* docs(rooster): resolve amplifier copper pattern and stage production review

* docs(rooster): record LED fuse and header review findings

* docs(rooster): specify capped vias and verify mask clearance

* docs(rooster): verify mask bridges and prepare exact RTC preorder

* fix(rooster): allow finished-hole tolerance at main display header

* fab(rooster): export checked header-fit candidates and rebind placements

* Bind prototype via process attachments to current fabrication files

* Define prototype stackup and record USB functional-test disposition

* Record updated main quote with current Gerbers and fill-cap stackup

* docs(rooster): refresh Beacon quote and first-power handoff

* docs(rooster): prepare exact placement review and external inventory

* docs(rooster): define immediate order gates and prototype power scope

* docs(rooster): compare stocked RTC alternatives and compatibility

* docs(rooster): compare RTC manufacturers and enclosure thermal limits

* docs(rooster): compare PCB manufacturing and assembly suppliers

* docs(rooster): stage Cube first and retain JLCPCB recommendation

* docs(rooster): re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
Parts:
- C35: LCSC# (none) -> C782172; MPN GRM188R61A106KAALD -> GRT188R61A106KE13D; Manufacturer (none) -> Murata Electronics
- C36, C37: LCSC# (none) -> C45000; Manufacturer (none) -> Murata Electronics
- J3: LCSC# (none) -> C5930350; Manufacturer (none) -> Samtec
- R54, R55, R56: LCSC# (none) -> C60491; Manufacturer (none) -> YAGEO
- U10: LCSC# (none) -> C2866750; Manufacturer (none) -> Texas Instruments
Changed lines of the file:
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@@
 		(property
 			"Datasheet"
-			"https://www.ti.com/lit/ds/symlink/tmux1511.pdf"
+			"https://www.ti.com/cn/lit/gpn/tmux1511"
 			(at 100.33 81.28 0)
 			(effects
@@
 		(pin
 			"14"
-))
+)
+	(property "Manufacturer" "Texas Instruments" (at 0 0 0) (effects (font (size 1.27 1.27)) (hide yes)))
+	(property "LCSC#" "C2866750" (at 0 0 0) (effects (font (size 1.27 1.27)) (hide yes))))
 	(wire
 		(pts
@@
 		(property
 			"Datasheet"
-			"https://www.hlktech.com/en/Goods-239.html"
+			"https://www.samtec.com/products/ssw-105-01-f-s"
 			(at 215.9 76.2 0)
 			(effects
@@
 		(pin
 			"5"
-))
+)
+	(property "Manufacturer" "Samtec" (at 0 0 0) (effects (font (size 1.27 1.27)) (hide yes)))
+	(property "LCSC#" "C5930350" (at 0 0 0) (effects (font (size 1.27 1.27)) (hide yes))))
 	(wire
 		(pts
@@
 		(property
 			"Datasheet"
-			""
+			"https://www.lcsc.com/datasheet/lcsc_datasheet_2304140030_YAGEO-RC0402FR-07100KL_C60491.pdf"
 			(at 43.18 111.76 0)
 			(effects
@@
 		(pin
 			"2"
-))
+)
+	(property "Manufacturer" "YAGEO" (at 0 0 0) (effects (font (size 1.27 1.27)) (hide yes)))
+	(property "LCSC#" "C60491" (at 0 0 0) (effects (font (size 1.27 1.27)) (hide yes))))
 	(wire
 		(pts
@@
 		(property
 			"Datasheet"
-			""
+			"https://www.lcsc.com/datasheet/lcsc_datasheet_2304140030_YAGEO-RC0402FR-07100KL_C60491.pdf"
 			(at 43.18 139.7 0)
 			(effects
@@
 		(pin
 			"2"
-))
+)
+	(property "Manufacturer" "YAGEO" (at 0 0 0) (effects (font (size 1.27 1.27)) (hide yes)))
+	(property "LCSC#" "C60491" (at 0 0 0) (effects (font (size 1.27 1.27)) (hide yes))))
 	(wire
 		(pts
@@
 		(property
 			"Datasheet"
-			""
+			"https://www.lcsc.com/datasheet/lcsc_datasheet_2304140030_YAGEO-RC0402FR-07100KL_C60491.pdf"
 			(at 93.98 139.7 0)
 			(effects
@@
 		(pin
 			"2"
-))
+)
+	(property "Manufacturer" "YAGEO" (at 0 0 0) (effects (font (size 1.27 1.27)) (hide yes)))
+	(property "LCSC#" "C60491" (at 0 0 0) (effects (font (size 1.27 1.27)) (hide yes))))
 	(wire
 		(pts
@@
 		(property
 			"Datasheet"
-			"https://datasheet.octopart.com/GRM188R61A106KAALD-Murata-datasheet-138742814.pdf"
+			"https://search.murata.co.jp/Ceramy/image/img/A01X/G101/ENG/GRT188R61A106KE13-01A.pdf"
 			(at 215.9 114.3 0)
 			(effects
@@
 		(property
 			"MPN"
-			"GRM188R61A106KAALD"
+			"GRT188R61A106KE13D"
 			(at 215.9 114.3 0)
 			(effects
@@
 				(font
 					(size 1.27 1.27))
-				(hide yes))))
+				(hide yes)))
+	(property "Manufacturer" "Murata Electronics" (at 0 0 0) (effects (font (size 1.27 1.27)) (hide yes)))
+	(property "LCSC#" "C782172" (at 0 0 0) (effects (font (size 1.27 1.27)) (hide yes))))
 	(wire
 		(pts
@@
 		(property
 			"Datasheet"
-			"https://www.murata.com/en-us/products/productdetail?partno=GRM188R71C104KA01D"
+			"https://wmsc.lcsc.com/wmsc/upload/file/pdf/v2/lcsc/1810311119_Murata-Electronics-GRM188R71C104KA01D_C45000.pdf"
 			(at 248.92 114.3 0)
 			(effects
@@
 				(font
 					(size 1.27 1.27))
-				(hide yes))))
+				(hide yes)))
+	(property "Manufacturer" "Murata Electronics" (at 0 0 0) (effects (font (size 1.27 1.27)) (hide yes)))
+	(property "LCSC#" "C45000" (at 0 0 0) (effects (font (size 1.27 1.27)) (hide yes))))
 	(wire
 		(pts
@@
 		(property
 			"Datasheet"
-			"https://www.murata.com/en-us/products/productdetail?partno=GRM188R71C104KA01D"
+			"https://wmsc.lcsc.com/wmsc/upload/file/pdf/v2/lcsc/1810311119_Murata-Electronics-GRM188R71C104KA01D_C45000.pdf"
 			(at 149.86 139.7 0)
 			(effects
@@
 				(font
 					(size 1.27 1.27))
-				(hide yes))))
+				(hide yes)))
+	(property "Manufacturer" "Murata Electronics" (at 0 0 0) (effects (font (size 1.27 1.27)) (hide yes)))
+	(property "LCSC#" "C45000" (at 0 0 0) (effects (font (size 1.27 1.27)) (hide yes))))
 	(hierarchical_label
 		"3v3"
